File: PlacaCuatroReles.kicad_sch (KiCad schematic)
At the start: 23 parts, among them J1 TBP01R1-508-02BE, J2 Conn_01x01_Pin, J3 Conn_01x01_Pin, J4 Conn_01x01_Pin, J5 Conn_01x01_Pin, J6 Conn_01x01_Pin, J7 Conn_01x01_Pin, J8 Conn_01x01_Pin, K1 SANYOU_SRD_Form_C, K2 SANYOU_SRD_Form_C, K3 SANYOU_SRD_Form_C, K4 SANYOU_SRD_Form_C

Commit message: Se agregó capa Silkscreen para señalizar las señales de acuerdo al diagrama de conexionado de la placa.
Other:
- note added: "+"
- note added: "-"
- note added: "Amarillo Sirena EVO"
- note added: "Blanco ZX8"
- note added: "Negativo Bastidor"
- note added: "Negativo Sirena"
- note added: "Negativo Sirena EVO"
- note added: "PGM4 Normal Abierto"
- note added: "Verde ZX8"
Changed lines of the file:
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@@
 		(comment 4 "Placa Cuatro Reles")
+	)
+	(text "PGM4 Normal Abierto"
+		(exclude_from_sim no)
+		(at 187.96 108.585 0)
+		(effects
+			(font
+				(size 2.54 2.54)
+			)
+		)
+	)
+	(text "Blanco ZX8"
+		(exclude_from_sim no)
+		(at 178.435 29.21 0)
+		(effects
+			(font
+				(size 2.54 2.54)
+			)
+		)
+	)
+	(text "Negativo Bastidor"
+		(exclude_from_sim no)
+		(at 184.15 67.945 0)
+		(effects
+			(font
+				(size 2.54 2.54)
+			)
+		)
+	)
+	(text "+"
+		(exclude_from_sim no)
+		(at 40.005 96.52 0)
+		(effects
+			(font
+				(size 2.54 2.54)
+			)
+		)
+	)
+	(text "Negativo Sirena\n"
+		(exclude_from_sim no)
+		(at 182.245 87.63 0)
+		(effects
+			(font
+				(size 2.54 2.54)
+			)
+		)
+	)
+	(text "-\n"
+		(exclude_from_sim no)
+		(at 40.005 100.965 0)
+		(effects
+			(font
+				(size 2.54 2.54)
+			)
+		)
+	)
+	(text "Amarillo Sirena EVO"
+		(exclude_from_sim no)
+		(at 186.69 149.86 0)
+		(effects
+			(font
+				(size 2.54 2.54)
+			)
+		)
+	)
+	(text "Negativo Sirena EVO\n"
+		(exclude_from_sim no)
+		(at 187.325 128.27 0)
+		(effects
+			(font
+				(size 2.54 2.54)
+			)
+		)
+	)
+	(text "Verde ZX8"
+		(exclude_from_sim no)
+		(at 176.53 49.53 0)
+		(effects
+			(font
+				(size 2.54 2.54)
+			)
+		)
 	)
 	(junction
